Commit message: worked on urdf

File: eeduro_delta_description/urdf/eeduro_delta.urdf (robot description, URDF)
Before this commit: robot eeduro_delta, 4 links, 3 joints
Links:
- added link link2_arm1, mass 0.002676077437253; visual mesh filename=package://eeduro_delta_description/meshes/link2_scaled.dae
- added link link3_0_arm1, mass 0.00303456300894497; visual mesh filename=package://eeduro_delta_description/meshes/link3_scaled.dae
- added link link3_1_arm1, mass 0.00303456300894497; visual mesh filename=package://eeduro_delta_description/meshes/link3_scaled.dae
- added link link4_arm1, mass 0.002676077437253; visual mesh filename=package://eeduro_delta_description/meshes/link2_scaled.dae
- link base_link: mass 1.0 -> 1.9
- link link1_arm1: mass 1 -> 0.01225732594264; geometry visual mesh filename=package://eeduro_delta_description/meshes/link1_scaled.dae
Joints:
- added joint joint1_arm1: type continuous, parent link1_arm1, child link2_arm1, origin xyz=0 0 0.05 rpy=0 0 0, axis 1 0 0
- added joint joint2_0_arm1: type continuous, parent link2_arm1, child link3_0_arm1, origin xyz=0.018 0 0 rpy=0 0 -1.570796327, axis 1 0 0
- added joint joint2_1_arm1: type continuous, parent link2_arm1, child link3_1_arm1, origin xyz=-0.018 0 0 rpy=0 0 -1.570796327, axis 1 0 0
- added joint joint3_0_arm1: type continuous, parent link3_0_arm1, child link4_arm1, origin xyz=0 0 0.1 rpy=0 0 0, axis 1 0 0

Commit message: finihed arm1 in urdf

File: eeduro_delta_description/urdf/eeduro_delta.urdf (robot description, URDF)
Before this commit: robot eeduro_delta, 8 links, 7 joints
Links:
- added link tool, mass 0.05741035631797; collision cylinder length=0.051 radius=0.007; visual mesh filename=package://eeduro_delta_description/meshes/tool_scaled.dae
Joints:
- added joint joint4_arm1: type continuous, parent link4_arm1, child tool, origin xyz=0 -0.018 0 rpy=-0.733038286 0 1.570796327, axis 1 0 0
- joint joint0_arm1: origin xyz=0 -0.052735026919 0.195 rpy=-2 0 3.141592654 -> xyz=0 -0.052735026919 0.195 rpy=-2.042035225 0 3.141592654
- joint joint1_arm1: origin xyz=0 0 0.05 rpy=0 0 0 -> xyz=0 0 0.05 rpy=-1.919862177 0 0
