Commit message: inertial-file rearanged content

File: eeduro_delta_description/urdf/eeduro_delta_inertial.urdf.xacro (robot description, xacro)
@@ -3,84 +3,81 @@
 	<xacro:macro name="base_inertial">
 		<inertial>
-			<origin xyz="-3.61483029333e-10 0.0127334577336 0.0879729092856" rpy="0 0 0"/>
+			<origin		xyz="	-3.61483029333e-10
+											 0.0127334577336
+											 0.0879729092856"
+								rpy="0 0 0"/>
 			<mass value="1.9"/>
-			<inertia  ixx="0.02085588597106"
-	              ixy="-1.660569664432e-10"
-	              ixz="-1.1398676896544e-10"
-	              iyy="0.02129590096144"
-	              iyz="0.0016993275934572"
-		            izz="0.019156198852616"/>
+			<inertia  ixx="0.02085588597106"			ixy="-1.660569664432e-10"		ixz="-1.1398676896544e-10"
+																						iyy="0.02129590096144"			iyz="0.0016993275934572"
+																																				izz="0.019156198852616"/>
 		</inertial>
 	</xacro:macro>
 	<xacro:macro name="motor_inertial">
 		<inertial>
-      <origin xyz="0 0 0" rpy="0 0 0"/>
+      <origin		xyz="0 0 0" rpy="0 0 0"/>
       <mass value="0.01"/>
-      <inertia	ixx="6.5e-8"
-								ixy="0"
-								ixz="0"
-								iyy="8.5e-8"
-								iyz="0"
-								izz="8.5e-8"/>
+      <inertia	ixx="6.5e-8"								ixy="0"											ixz="0"
+																						iyy="8.5e-8"								iyz="0"
+																																				izz="8.5e-8"/>
     </inertial>
 	</xacro:macro>
 	<xacro:macro name="link1_inertial">
 		<inertial>
-	    <origin xyz="-0.000667579518792749 4.24024711964181e-05 0.0237382053187016" rpy="0 0 0"/>
+	    <origin		xyz="	-0.000667579518792749
+											 4.24024711964181e-05
+											 0.0237382053187016"
+								rpy="0 0 0"/>
 	    <mass value="0.01225732594264"/>
-	    <inertia  ixx="3.9170528247202e-06"
-	              ixy="6.88244852580979e-11"
-	              ixz="-4.1443351708254e-08"
-	              iyy="3.81032017743918e-06"
-	              iyz="1.23377194660718e-08"
-	              izz="1.78939838618822e-07"/>
+	    <inertia  ixx="3.9170528247202e-06"		ixy="6.88244852580979e-11"	ixz="-4.1443351708254e-08"
+																						iyy="3.81032017743918e-06"	iyz="1.23377194660718e-08"
+																																				izz="1.78939838618822e-07"/>
 	  </inertial>
 	</xacro:macro>
 	<xacro:macro name="link2_inertial">
 		<inertial>
-	    <origin xyz="-4.65883028011777e-16 0.000173858781653159 5.67176538207829e-17" rpy="0 0 0"/>
+	    <origin		xyz="	-4.65883028011777e-16
+											 0.000173858781653159
+											 5.67176538207829e-17"
+								rpy="0 0 0"/>
 	    <mass value="0.002676077437253"/>
-	    <inertia  ixx="2.12767184543771e-08"
-	              ixy="-5.53089204125579e-22"
-	              ixz="-3.40282030897929e-10"
-	              iyy="5.08472734636316e-07"
-	              iyz="1.63502204451954e-23"
-	              izz="5.19396055186747e-07"/>
+	    <inertia  ixx="2.12767184543771e-08"	ixy="-5.53089204125579e-22"	ixz="-3.40282030897929e-10"
+																						iyy="5.08472734636316e-07"	iyz="1.63502204451954e-23"
+																																				izz="5.19396055186747e-07"/>
 	  </inertial>
 	</xacro:macro>
 	<xacro:macro name="link3_inertial">
 		<inertial>
-	    <origin xyz="4.79435653399733e-15 5.05515762210611e-15 0.05" rpy="0 0 0"/>
+	    <origin		xyz="	4.79435653399733e-15
+											5.05515762210611e-15
+											0.05"
+								rpy="0 0 0"/>
 	    <mass value="0.00303456300894497"/>
-	    <inertia  ixx="3.21114513230401e-06"
-	              ixy="-1.39831896086795e-22"
-	              ixz="-1.65818121965606e-19"
-	              iyy="3.20896476471281e-06"
-	              iyz="-7.25104237772119e-20"
-	              izz="5.81686125403351e-09"/>
+	    <inertia  ixx="3.21114513230401e-06"	ixy="-1.39831896086795e-22"	ixz="-1.65818121965606e-19"
+																						iyy="3.20896476471281e-06"	iyz="-7.25104237772119e-20"
+																																				izz="5.81686125403351e-09"/>
 	  </inertial>
 	</xacro:macro>
 	<xacro:macro name="link4_inertial">
 		<inertial>
-	    <origin xyz="-0.00017385878165316 -0.0179999999999995 -5.56154717015503e-17" rpy="0 0 0"/>
+	    <origin		xyz="	-0.00017385878165316
+											-0.0179999999999995
+											-5.56154717015503e-17"
+								rpy="0 0 0"/>
 	    <mass value="0.002676077437253"/>
-	    <inertia  ixx="5.08472734636316e-07"
-	              ixy="-5.82921356214306e-22"
-	              ixz="1.63293841801982e-23"
-	              iyy="2.12767184543771e-08"
-	              iyz="-3.40282030897868e-10"
-	              izz="5.19396055186747e-07"/>
+	    <inertia  ixx="5.08472734636316e-07"	ixy="-5.82921356214306e-22"	ixz="1.63293841801982e-23"
+																						iyy="2.12767184543771e-08"	iyz="-3.40282030897868e-10"
+																																				izz="5.19396055186747e-07"/>
 	  </inertial>
 	</xacro:macro>
 	<xacro:macro name="tool_inertial">
 		<inertial>
-	    <origin xyz="2.59861008225168e-05 0.00192804788388403 0.022995128907788" rpy="0 0 0"/>
+	    <origin		xyz="	2.59861008225168e-05
+											0.00192804788388403
+											0.022995128907788"
+								rpy="0 0 0"/>
 	    <mass value="0.05741035631797"/>
-	    <inertia  ixx="1.98534599648007e-05"
-	              ixy="-5.03744139689366e-09"
-	              ixz="8.28383830393447e-10"
-	              iyy="5.51924419052098e-06"
-	              iyz="1.3955126250812e-08"
-	              izz="1.98271230263828e-05"/>
+	    <inertia  ixx="1.98534599648007e-05"	ixy="-5.03744139689366e-09"	ixz="8.28383830393447e-10"
+																						iyy="5.51924419052098e-06"	iyz="1.3955126250812e-08"
+																																				izz="1.98271230263828e-05"/>
 	  </inertial>
 	</xacro:macro>
