Commit message: xacro: added macro for arm (only motor in macro)

File: eeduro_delta_description/urdf/eeduro_delta.urdf.xacro (robot description, xacro)
@@ -24,17 +24,24 @@
 			</geometry>
 		</collision>
-		<xacro:base_link_inertial/>
+		<xacro:base_inertial/>
 	</link>
-<!--
-  <inertial>
-    <origin xyz="-3.61483029333e-10 0.0127334577336 0.0879729092856" rpy="0 0 0"/>
-    <mass value="1.9"/>
-    <inertia  ixx="0.02085588597106"
-              ixy="-1.660569664432e-10"
-              ixz="-1.1398676896544e-10"
-              iyy="0.02129590096144"
-              iyz="0.0016993275934572"
-              izz="0.019156198852616"/>
-  </inertial>
--->
+	<xacro:delta_arm parent="base_link" arm_nr="1"/>
+	<xacro:macro name="delta_arm" params="parent arm_nr">
+		<joint name="arm${arm_nr}_joint_motor" type="continuous">
+		  <parent link="${parent}"/>
+		  <child link="arm${arm_nr}_motor"/>
+		  <origin xyz="0.04 -0.052735026919 0.195" rpy="-1.570796327 0 3.141592654"/>
+		  <axis xyz="1 0 0"/>
+		  <dynamics damping="0.0000001"/>
+		</joint>
+		<link name="arm${arm_nr}_motor">
+	  <visual>
+	    <origin xyz="0 0 0" rpy="0 1.570796327 0"/>
+	    <geometry>
+	      <cylinder radius="0.006" length="0.018"/>
+	    </geometry>
+	  </visual>
+		<xacro:motor_inertial/>
+		</link>
+	</xacro:macro>
 </robot>

File: eeduro_delta_description/urdf/eeduro_delta_inertial.urdf.xacro (robot description, xacro)
@@ -1,5 +1,5 @@
 <?xml version="1.0"?>
 <robot name="eeduro_delta" xmlns:xacro="http://www.ros.org/wiki/xacro">
-	<xacro:macro name="base_link_inertial">
+	<xacro:macro name="base_inertial">
 		<inertial>
 			<origin xyz="-3.61483029333e-10 0.0127334577336 0.0879729092856" rpy="0 0 0"/>
@@ -13,3 +13,10 @@
 		</inertial>
 	</xacro:macro>
+	<xacro:macro name="motor_inertial">
+		<inertial>
+      <origin xyz="0 0 0" rpy="0 0 0"/>
+      <mass value="0.01"/>
+      <inertia ixx="6.5e-8" ixy="0" ixz="0" iyy="8.5e-8" iyz="0" izz="8.5e-8"/>
+    </inertial>
+	</xacro:macro>
 </robot>

Commit message: xacro: arm modeled till joint3

File: eeduro_delta_description/urdf/eeduro_delta.urdf.xacro (robot description, xacro)
@@ -1,4 +1,4 @@
 <?xml version="1.0"?>
-<robot name="eeduro_delta" xmlns:xacro="http://ww.ros.org/wiki/xacro">
+<robot name="eeduro_delta" xmlns:xacro="http://www.ros.org/wiki/xacro">
 	<xacro:property name="pi" value="3.1415926535897931"/>
 	<xacro:include filename="$(find eeduro_delta_description)/urdf/eeduro_delta_inertial.urdf.xacro"/>
@@ -28,5 +28,5 @@
 	<xacro:delta_arm parent="base_link" arm_nr="1"/>
 	<xacro:macro name="delta_arm" params="parent arm_nr">
-		<joint name="arm${arm_nr}_joint_motor" type="continuous">
+		<joint name="arm${arm_nr}_motor_joint" type="continuous">
 		  <parent link="${parent}"/>
 		  <child link="arm${arm_nr}_motor"/>
@@ -44,4 +44,72 @@
 		<xacro:motor_inertial/>
 		</link>
+		<joint name="arm${arm_nr}_joint0" type="continuous">
+		  <parent link="${parent}"/>
+		  <child link="arm${arm_nr}_link1"/>
+		  <!-- callculation X: 0  Y: -70.23..+17.5  Z: 210-15 -->
+		  <origin xyz="0 -0.052735026919 0.195" rpy="-2.042035225 0 3.141592654"/>
+		  <axis xyz="1 0 0"/>
+		  <dynamics damping="0.0001"/>
+		</joint>
+		<link name="arm${arm_nr}_link1">
+		  <visual>
+		    <origin xyz="0 0 0" rpy="0 0 0"/>
+		    <geometry>
+		      <!--<box size="0.01 0.01  0.06"/>-->
+		      <mesh filename="package://eeduro_delta_description/meshes/link1_scaled.dae"/>
+		    </geometry>
+		  </visual>
+			<xacro:link1_inertial/>
+		</link>
+		<gazebo>
+		  <joint name="arm${arm_nr}_gearbox" type="gearbox">
+		    <parent>arm${arm_nr}_motor</parent>
+		    <child>arm${arm_nr}_link1</child>
+		    <gearbox_reference_body>${parent}</gearbox_reference_body>
+		    <gearbox_ratio>-0.013176411</gearbox_ratio>
+		    <axis>
+		      <xyz>1 0 0</xyz>
+		    </axis>
+		    <axis2>
+		      <xyz>1 0 0</xyz>
+		    </axis2>
+		  </joint>
+		</gazebo>
+		<joint name="arm${arm_nr}_joint1" type="continuous">
+		  <parent link="arm${arm_nr}_link1"/>
+		  <child link="arm${arm_nr}_link2"/>
+		  <origin xyz="0 0 0.05" rpy="-1.919862177 0 0"/>
+		  <axis xyz="1 0 0"/>
+		  <dynamics damping="0.00001"/>
+		</joint>
+		<link name="arm${arm_nr}_link2">
+		  <visual>
+		    <origin xyz="0 0 0" rpy="0 0 0"/>
+		    <geometry>
+		      <mesh filename="package://eeduro_delta_description/meshes/link2_scaled.dae"/>
+		    </geometry>
+		  </visual>
+			<xacro:link2_inertial/>
+		</link>
+		<xacro:link3_with_joint arm_nr="${arm_nr}" suffix=".1" sign="+"/>
+		<xacro:link3_with_joint arm_nr="${arm_nr}" suffix=".2" sign="-"/>
+	</xacro:macro>
+	<xacro:macro name="link3_with_joint" params="arm_nr suffix sign">
+		<joint name="arm${arm_nr}_joint2${suffix}" type="continuous">
+		  <parent link="arm${arm_nr}_link2"/>
+		  <child link="arm${arm_nr}_link3${suffix}"/>
+		  <origin xyz="${sign}0.018 0 0" rpy="0 0 -1.570796327"/>
+		  <axis xyz="1 0 0"/>
+		  <dynamics damping="0.00001"/>
+		</joint>
+		<link name="arm${arm_nr}_link3${suffix}">
+		  <visual>
+		    <origin xyz="0 0 0" rpy="0 0 0"/>
+		    <geometry>
+		      <mesh filename="package://eeduro_delta_description/meshes/link3_scaled.dae"/>
+		    </geometry>
+		  </visual>
+			<xacro:link3_inertial/>
+		</link>
 	</xacro:macro>
 </robot>

File: eeduro_delta_description/urdf/eeduro_delta_inertial.urdf.xacro (robot description, xacro)
@@ -10,5 +10,5 @@
 	              iyy="0.02129590096144"
 	              iyz="0.0016993275934572"
-	             izz="0.019156198852616"/>
+		            izz="0.019156198852616"/>
 		</inertial>
 	</xacro:macro>
@@ -20,3 +20,39 @@
     </inertial>
 	</xacro:macro>
+	<xacro:macro name="link1_inertial">
+		<inertial>
+	    <origin xyz="-0.000667579518792749 4.24024711964181e-05 0.0237382053187016" rpy="0 0 0"/>
+	    <mass value="0.01225732594264"/>
+	    <inertia  ixx="3.9170528247202e-06"
+	              ixy="6.88244852580979e-11"
+	              ixz="-4.1443351708254e-08"
+	              iyy="3.81032017743918e-06"
+	              iyz="1.23377194660718e-08"
+	              izz="1.78939838618822e-07"/>
+	  </inertial>
+	</xacro:macro>
+	<xacro:macro name="link2_inertial">
+		<inertial>
+	    <origin xyz="-4.65883028011777e-16 0.000173858781653159 5.67176538207829e-17" rpy="0 0 0"/>
+	    <mass value="0.002676077437253"/>
+	    <inertia  ixx="2.12767184543771e-08"
+	              ixy="-5.53089204125579e-22"
+	              ixz="-3.40282030897929e-10"
+	              iyy="5.08472734636316e-07"
+	              iyz="1.63502204451954e-23"
+	              izz="5.19396055186747e-07"/>
+	  </inertial>
+	</xacro:macro>
+	<xacro:macro name="link3_inertial">
+		<inertial>
+	    <origin xyz="4.79435653399733e-15 5.05515762210611e-15 0.05" rpy="0 0 0"/>
+	    <mass value="0.00303456300894497"/>
+	    <inertia  ixx="3.21114513230401e-06"
+	              ixy="-1.39831896086795e-22"
+	              ixz="-1.65818121965606e-19"
+	              iyy="3.20896476471281e-06"
+	              iyz="-7.25104237772119e-20"
+	              izz="5.81686125403351e-09"/>
+	  </inertial>
+	</xacro:macro>
 </robot>

Commit message: xacro: added link4 and joints to close kinematic chain

File: eeduro_delta_description/urdf/eeduro_delta.urdf.xacro (robot description, xacro)
@@ -92,8 +92,17 @@
 			<xacro:link2_inertial/>
 		</link>
-		<xacro:link3_with_joint arm_nr="${arm_nr}" suffix=".1" sign="+"/>
-		<xacro:link3_with_joint arm_nr="${arm_nr}" suffix=".2" sign="-"/>
+		<xacro:link3_with_joint arm_nr="${arm_nr}" suffix="_1" sign="+" joint3_type="urdf"/>
+		<xacro:link3_with_joint arm_nr="${arm_nr}" suffix=".2" sign="-" joint3_type="sdf"/>
+		<link name="arm${arm_nr}_link4">
+		  <visual>
+		    <origin xyz="0 -0.018 0" rpy="0 0 1.570796327"/>
+		    <geometry>
+		      <mesh filename="package://eeduro_delta_description/meshes/link2_scaled.dae"/>
+		    </geometry>
+		  </visual>
+			<xacro:link4_inertial/>
+		</link>
 	</xacro:macro>
-	<xacro:macro name="link3_with_joint" params="arm_nr suffix sign">
+	<xacro:macro name="link3_with_joint" params="arm_nr suffix sign joint3_type">
 		<joint name="arm${arm_nr}_joint2${suffix}" type="continuous">
 		  <parent link="arm${arm_nr}_link2"/>
@@ -112,4 +121,34 @@
 			<xacro:link3_inertial/>
 		</link>
+		<xacro:element xacro:name="joint3_${joint3_type}" arm_nr="${arm_nr}" suffix="${suffix}"/>
 	</xacro:macro>
+	<xacro:macro name="joint3_urdf" params="arm_nr suffix">
+			<joint name="arm${arm_nr}_link3${suffix}" type="continuous">
+			  <parent link="arm${arm_nr}_link3${suffix}"/>
+			  <child link="arm${arm_nr}_link4"/>
+			  <origin xyz="0 0 0.1" rpy="0 0 0"/>
+			  <axis xyz="1 0 0"/>
+			  <dynamics damping="0.00001"/>
+			</joint>
+	</xacro:macro>
+	<xacro:macro name="joint3_sdf" params="arm_nr suffix">
+		<gazebo>
+			<joint name="arm${arm_nr}_joint3${suffix}" type="revolute">
+			  <child>arm${arm_nr}_link4</child>
+			  <parent>arm${arm_nr}_link3${suffix}</parent>
+			  <pose>0 -0.036 0 0 0 0</pose>
+			  <axis>
+			    <use_parent_model_frame>false</use_parent_model_frame>
+			    <xyz>1 0 0</xyz>
+			    <limit>
+			      <lower>-1e+16</lower>
+			      <upper>1e+16</upper>
+			    </limit>
+			    <dynamics>
+			      <damping>0.00001</damping>
+			    </dynamics>
+			  </axis>
+			</joint>
+		</gazebo>
+  </xacro:macro>
 </robot>

File: eeduro_delta_description/urdf/eeduro_delta_inertial.urdf.xacro (robot description, xacro)
@@ -56,3 +56,15 @@
 	  </inertial>
 	</xacro:macro>
+	<xacro:macro name="link4_inertial">
+		<inertial>
+	    <origin xyz="-0.00017385878165316 -0.0179999999999995 -5.56154717015503e-17" rpy="0 0 0"/>
+	    <mass value="0.002676077437253"/>
+	    <inertia  ixx="5.08472734636316e-07"
+	              ixy="-5.82921356214306e-22"
+	              ixz="1.63293841801982e-23"
+	              iyy="2.12767184543771e-08"
+	              iyz="-3.40282030897868e-10"
+	              izz="5.19396055186747e-07"/>
+	  </inertial>
+	</xacro:macro>
 </robot>

Commit message: xacro: added tool

File: eeduro_delta_description/urdf/eeduro_delta.urdf.xacro (robot description, xacro)
@@ -103,4 +103,11 @@
 			<xacro:link4_inertial/>
 		</link>
+		<joint name="arm${arm_nr}_joint4" type="continuous">
+		  <parent link="arm${arm_nr}_link4"/>
+		  <child link="tool"/>
+		  <origin xyz="0 -0.018 0" rpy="-0.733038286 0 1.570796327"/>
+		  <axis xyz="1 0 0"/>
+		  <dynamics damping="0.00001"/>
+		</joint>
 	</xacro:macro>
 	<xacro:macro name="link3_with_joint" params="arm_nr suffix sign joint3_type">
@@ -152,3 +159,24 @@
 		</gazebo>
   </xacro:macro>
+	<link name="tool">
+	  <visual>
+	    <origin xyz="0 0 0" rpy="0 0 0"/>
+	    <geometry>
+	      <mesh filename="package://eeduro_delta_description/meshes/tool_scaled.dae"/>
+	    </geometry>
+	  </visual>
+	  <collision>
+	    <origin xyz="0 0 0.023" rpy="1.570796327 0 0"/>
+	    <geometry>
+	      <cylinder radius="0.007" length="0.051"/>
+	    </geometry>
+	  </collision>
+		<xacro:tool_inertial/>
+	</link>
+	<gazebo reference="base_link">
+	  <selfCollide>true</selfCollide>
+	</gazebo>
+	<gazebo reference="tool">
+	  <selfCollide>true</selfCollide>
+	</gazebo>
 </robot>

File: eeduro_delta_description/urdf/eeduro_delta_inertial.urdf.xacro (robot description, xacro)
@@ -68,3 +68,15 @@
 	  </inertial>
 	</xacro:macro>
+	<xacro:macro name="tool_inertial">
+		<inertial>
+	    <origin xyz="2.59861008225168e-05 0.00192804788388403 0.022995128907788" rpy="0 0 0"/>
+	    <mass value="0.05741035631797"/>
+	    <inertia  ixx="1.98534599648007e-05"
+	              ixy="-5.03744139689366e-09"
+	              ixz="8.28383830393447e-10"
+	              iyy="5.51924419052098e-06"
+	              iyz="1.3955126250812e-08"
+	              izz="1.98271230263828e-05"/>
+	  </inertial>
+	</xacro:macro>
 </robot>

Commit message: xacro: replaced hard coded angles with expressions

File: eeduro_delta_description/urdf/eeduro_delta.urdf.xacro (robot description, xacro)
@@ -27,9 +27,30 @@
 	</link>
 	<xacro:delta_arm parent="base_link" arm_nr="1"/>
+	<link name="tool">
+	  <visual>
+	    <origin xyz="0 0 0" rpy="0 0 0"/>
+	    <geometry>
+	      <mesh filename="package://eeduro_delta_description/meshes/tool_scaled.dae"/>
+	    </geometry>
+	  </visual>
+	  <collision>
+	    <origin xyz="0 0 0.023" rpy="${pi/2} 0 0"/>
+	    <geometry>
+	      <cylinder radius="0.007" length="0.051"/>
+	    </geometry>
+	  </collision>
+		<xacro:tool_inertial/>
+	</link>
+	<gazebo reference="base_link">
+	  <selfCollide>true</selfCollide>
+	</gazebo>
+	<gazebo reference="tool">
+	  <selfCollide>true</selfCollide>
+	</gazebo>
 	<xacro:macro name="delta_arm" params="parent arm_nr">
 		<joint name="arm${arm_nr}_motor_joint" type="continuous">
 		  <parent link="${parent}"/>
 		  <child link="arm${arm_nr}_motor"/>
-		  <origin xyz="0.04 -0.052735026919 0.195" rpy="-1.570796327 0 3.141592654"/>
+		  <origin xyz="0.04 -0.052735026919 0.195" rpy="${-pi/2} 0 ${pi}"/>
 		  <axis xyz="1 0 0"/>
 		  <dynamics damping="0.0000001"/>
@@ -37,5 +58,5 @@
 		<link name="arm${arm_nr}_motor">
 	  <visual>
-	    <origin xyz="0 0 0" rpy="0 1.570796327 0"/>
+	    <origin xyz="0 0 0" rpy="0 ${pi/2} 0"/>
 	    <geometry>
 	      <cylinder radius="0.006" length="0.018"/>
@@ -48,5 +69,5 @@
 		  <child link="arm${arm_nr}_link1"/>
 		  <!-- callculation X: 0  Y: -70.23..+17.5  Z: 210-15 -->
-		  <origin xyz="0 -0.052735026919 0.195" rpy="-2.042035225 0 3.141592654"/>
+		  <origin xyz="0 -0.052735026919 0.195" rpy="${(-90-27)/180 *pi} 0 ${pi}"/>
 		  <axis xyz="1 0 0"/>
 		  <dynamics damping="0.0001"/>
@@ -79,5 +100,5 @@
 		  <parent link="arm${arm_nr}_link1"/>
 		  <child link="arm${arm_nr}_link2"/>
-		  <origin xyz="0 0 0.05" rpy="-1.919862177 0 0"/>
+		  <origin xyz="0 0 0.05" rpy="${(-110)/180*pi} 0 0"/>
 		  <axis xyz="1 0 0"/>
 		  <dynamics damping="0.00001"/>
@@ -96,5 +117,5 @@
 		<link name="arm${arm_nr}_link4">
 		  <visual>
-		    <origin xyz="0 -0.018 0" rpy="0 0 1.570796327"/>
+		    <origin xyz="0 -0.018 0" rpy="0 0 ${pi/2}"/>
 		    <geometry>
 		      <mesh filename="package://eeduro_delta_description/meshes/link2_scaled.dae"/>
@@ -106,5 +127,5 @@
 		  <parent link="arm${arm_nr}_link4"/>
 		  <child link="tool"/>
-		  <origin xyz="0 -0.018 0" rpy="-0.733038286 0 1.570796327"/>
+		  <origin xyz="0 -0.018 0" rpy="${(-43)/180*pi} 0 ${pi/2}"/>
 		  <axis xyz="1 0 0"/>
 		  <dynamics damping="0.00001"/>
@@ -115,5 +136,5 @@
 		  <parent link="arm${arm_nr}_link2"/>
 		  <child link="arm${arm_nr}_link3${suffix}"/>
-		  <origin xyz="${sign}0.018 0 0" rpy="0 0 -1.570796327"/>
+		  <origin xyz="${sign}0.018 0 0" rpy="0 0 ${-pi/2}"/>
 		  <axis xyz="1 0 0"/>
 		  <dynamics damping="0.00001"/>
@@ -159,24 +180,3 @@
 		</gazebo>
   </xacro:macro>
-	<link name="tool">
-	  <visual>
-	    <origin xyz="0 0 0" rpy="0 0 0"/>
-	    <geometry>
-	      <mesh filename="package://eeduro_delta_description/meshes/tool_scaled.dae"/>
-	    </geometry>
-	  </visual>
-	  <collision>
-	    <origin xyz="0 0 0.023" rpy="1.570796327 0 0"/>
-	    <geometry>
-	      <cylinder radius="0.007" length="0.051"/>
-	    </geometry>
-	  </collision>
-		<xacro:tool_inertial/>
-	</link>
-	<gazebo reference="base_link">
-	  <selfCollide>true</selfCollide>
-	</gazebo>
-	<gazebo reference="tool">
-	  <selfCollide>true</selfCollide>
-	</gazebo>
 </robot>

File: eeduro_delta_description/urdf/eeduro_delta_inertial.urdf.xacro (robot description, xacro)
@@ -17,5 +17,10 @@
       <origin xyz="0 0 0" rpy="0 0 0"/>
       <mass value="0.01"/>
-      <inertia ixx="6.5e-8" ixy="0" ixz="0" iyy="8.5e-8" iyz="0" izz="8.5e-8"/>
+      <inertia	ixx="6.5e-8"
+								ixy="0"
+								ixz="0"
+								iyy="8.5e-8"
+								iyz="0"
+								izz="8.5e-8"/>
     </inertial>
 	</xacro:macro>

Commit message: xacro: move angle definition to macro input

File: eeduro_delta_description/urdf/eeduro_delta.urdf.xacro (robot description, xacro)
@@ -26,5 +26,12 @@
 		<xacro:base_inertial/>
 	</link>
-	<xacro:delta_arm parent="base_link" arm_nr="1"/>
+	<xacro:delta_arm
+		parent="base_link"
+		arm_end_child="tool"
+		arm_nr="1"
+		joint4_type="urdf"
+		angle1="${(-90-27)/180 *pi}"
+		angle2="${(-110)/180*pi}"
+		angle3="${(-43)/180*pi}"/>
 	<link name="tool">
 	  <visual>
@@ -48,5 +55,5 @@
 	  <selfCollide>true</selfCollide>
 	</gazebo>
-	<xacro:macro name="delta_arm" params="parent arm_nr">
+	<xacro:macro name="delta_arm" params="parent arm_end_child arm_nr joint4_type angle1 angle2 angle3">
 		<joint name="arm${arm_nr}_motor_joint" type="continuous">
 		  <parent link="${parent}"/>
@@ -69,5 +76,5 @@
 		  <child link="arm${arm_nr}_link1"/>
 		  <!-- callculation X: 0  Y: -70.23..+17.5  Z: 210-15 -->
-		  <origin xyz="0 -0.052735026919 0.195" rpy="${(-90-27)/180 *pi} 0 ${pi}"/>
+		  <origin xyz="0 -0.052735026919 0.195" rpy="${angle1} 0 ${pi}"/>
 		  <axis xyz="1 0 0"/>
 		  <dynamics damping="0.0001"/>
@@ -77,5 +84,4 @@
 		    <origin xyz="0 0 0" rpy="0 0 0"/>
 		    <geometry>
-		      <!--<box size="0.01 0.01  0.06"/>-->
 		      <mesh filename="package://eeduro_delta_description/meshes/link1_scaled.dae"/>
 		    </geometry>
@@ -100,5 +106,5 @@
 		  <parent link="arm${arm_nr}_link1"/>
 		  <child link="arm${arm_nr}_link2"/>
-		  <origin xyz="0 0 0.05" rpy="${(-110)/180*pi} 0 0"/>
+		  <origin xyz="0 0 0.05" rpy="${angle2} 0 0"/>
 		  <axis xyz="1 0 0"/>
 		  <dynamics damping="0.00001"/>
@@ -124,11 +130,5 @@
 			<xacro:link4_inertial/>
 		</link>
-		<joint name="arm${arm_nr}_joint4" type="continuous">
-		  <parent link="arm${arm_nr}_link4"/>
-		  <child link="tool"/>
-		  <origin xyz="0 -0.018 0" rpy="${(-43)/180*pi} 0 ${pi/2}"/>
-		  <axis xyz="1 0 0"/>
-		  <dynamics damping="0.00001"/>
-		</joint>
+		<xacro:element xacro:name="joint4_${joint4_type}" arm_nr="${arm_nr}" child="${arm_end_child}" angle="${angle3}"/>
 	</xacro:macro>
 	<xacro:macro name="link3_with_joint" params="arm_nr suffix sign joint3_type">
@@ -180,3 +180,12 @@
 		</gazebo>
   </xacro:macro>
+	<xacro:macro name="joint4_urdf" params="arm_nr child angle">
+		<joint name="arm${arm_nr}_joint4" type="continuous">
+		  <parent link="arm${arm_nr}_link4"/>
+		  <child link="${child}"/>
+		  <origin xyz="0 -0.018 0" rpy="${angle} 0 ${pi/2}"/>
+		  <axis xyz="1 0 0"/>
+		  <dynamics damping="0.00001"/>
+		</joint>
+	</xacro:macro>
 </robot>

Commit message: changed how poition and orientation for arm is defined

File: eeduro_delta_description/urdf/eeduro_delta.urdf.xacro (robot description, xacro)
@@ -1,5 +1,7 @@
 <?xml version="1.0"?>
 <robot name="eeduro_delta" xmlns:xacro="http://www.ros.org/wiki/xacro">
-	<xacro:property name="pi" value="3.1415926535897931"/>
+	<!-- <xacro:property name="pi" value="3.1415926535897931"/> -->
+	<xacro:property name="dist_origin2arm_z" value="0.21"/>
+	<xacro:property name="dist_origin2arm_xy_plane" value="${0.1/sqrt(3) -0.005}"/>
 	<xacro:include filename="$(find eeduro_delta_description)/urdf/eeduro_delta_inertial.urdf.xacro"/>
 	<!--<xacro:include filename="$(find eeduro_delta_description)/urdf/eeduro_delta.gazebo.xacro"/>-->
@@ -31,7 +33,11 @@
 		arm_nr="1"
 		joint4_type="urdf"
-		angle1="${(-90-27)/180 *pi}"
+		angle1="${(-27)/180 *pi}"
 		angle2="${-0.8373228137897161 -(90-27)/180*pi}"
-		angle3="${-pi/2 + 0.8373228137897161}"/>
+		angle3="${-pi/2 + 0.8373228137897161}"
+		dist_xy="${dist_origin2arm_xy_plane}"
+		x="0"		y="0"		z="${dist_origin2arm_z}"
+		roll="0"		pitch="0"		yaw="${-pi/2}"
+	/>
 	<link name="tool">
 	  <visual>
@@ -55,9 +61,10 @@
 	  <selfCollide>true</selfCollide>
 	</gazebo>
-	<xacro:macro name="delta_arm" params="parent arm_end_child arm_nr joint4_type angle1 angle2 angle3">
+	<!-- x y z are the center of the robot, in the high:of the mounting-points for the arms -->
+	<xacro:macro name="delta_arm" params="parent arm_end_child arm_nr joint4_type angle1 angle2 angle3 dist_xy x y z roll pitch yaw">
 		<joint name="arm${arm_nr}_motor_joint" type="continuous">
 		  <parent link="${parent}"/>
 		  <child link="arm${arm_nr}_motor"/>
-		  <origin xyz="0.04 -0.052735026919 0.195" rpy="${-pi/2} 0 ${pi}"/>
+		  <origin xyz="${x +cos(yaw)*dist_xy -sin(yaw)*(0.04)} ${y +sin(yaw)*dist_xy +cos(yaw)*(0.04)} ${z -0.015}" rpy="${roll -pi/2} ${pitch} ${yaw -pi/2}"/>
 		  <axis xyz="1 0 0"/>
 		  <dynamics damping="0.0000001"/>
@@ -76,5 +83,5 @@
 		  <child link="arm${arm_nr}_link1"/>
 		  <!-- callculation X: 0  Y: -70.23..+17.5  Z: 210-15 -->
-		  <origin xyz="0 -0.052735026919 0.195" rpy="${angle1} 0 ${pi}"/>
+		  <origin xyz="${x +cos(yaw)*dist_xy} ${y +sin(yaw)*dist_xy}  ${z -0.015}" rpy="${roll -pi/2  +angle1} ${pitch} ${yaw -pi/2}"/>
 		  <axis xyz="1 0 0"/>
 		  <dynamics damping="0.0001"/>
@@ -120,5 +127,5 @@
 		</link>
 		<xacro:link3_with_joint arm_nr="${arm_nr}" suffix="_1" sign="+" joint3_type="urdf"/>
-		<xacro:link3_with_joint arm_nr="${arm_nr}" suffix=".2" sign="-" joint3_type="sdf"/>
+		<xacro:link3_with_joint arm_nr="${arm_nr}" suffix="_2" sign="-" joint3_type="sdf"/>
 		<link name="arm${arm_nr}_link4">
 		  <visual>

Commit message: xacro: added arm2 and arm3, some bug-fixes for sdf-joints

File: eeduro_delta_description/urdf/eeduro_delta.urdf.xacro (robot description, xacro)
@@ -40,4 +40,28 @@
 		roll="0"		pitch="0"		yaw="${-pi/2}"
 	/>
+	<xacro:delta_arm
+    parent="base_link"
+    arm_end_child="tool"
+    arm_nr="2"
+    joint4_type="sdf"
+    angle1="${(-27)/180 *pi}"
+    angle2="${-0.8373228137897161 -(90-27)/180*pi}"
+    angle3="${-pi/2 + 0.8373228137897161}"
+    dist_xy="${dist_origin2arm_xy_plane}"
+    x="0"   y="0"   z="${dist_origin2arm_z}"
+    roll="0"    pitch="0"   yaw="${pi/6}"
+  />
+	<xacro:delta_arm
+    parent="base_link"
+    arm_end_child="tool"
+    arm_nr="3"
+    joint4_type="sdf"
+    angle1="${(-27)/180 *pi}"
+    angle2="${-0.8373228137897161 -(90-27)/180*pi}"
+    angle3="${-pi/2 + 0.8373228137897161}"
+    dist_xy="${dist_origin2arm_xy_plane}"
+    x="0"   y="0"   z="${dist_origin2arm_z}"
+    roll="0"    pitch="0"   yaw="${5*pi/6}"
+  />
 	<link name="tool">
 	  <visual>
@@ -103,7 +127,9 @@
 		    <gearbox_ratio>-0.013176411</gearbox_ratio>
 		    <axis>
+					<use_parent_model_frame>false</use_parent_model_frame>
 		      <xyz>1 0 0</xyz>
 		    </axis>
 		    <axis2>
+					<use_parent_model_frame>false</use_parent_model_frame>
 		      <xyz>1 0 0</xyz>
 		    </axis2>
@@ -196,3 +222,23 @@
 		</joint>
 	</xacro:macro>
+  <xacro:macro name="joint4_sdf" params="arm_nr child angle">
+    <gazebo>
+			<joint name="arm${arm_nr}_joint4" type="revolute">
+	      <parent>${child}</parent>
+	      <child>arm${arm_nr}_link4</child>
+	      <pose>0 -0.018 0 ${angle} 0 ${pi/2}</pose>
+				<axis>
+          <use_parent_model_frame>false</use_parent_model_frame>
+          <xyz>1 0 0</xyz>
+          <limit>
+            <lower>-1e+16</lower>
+            <upper>1e+16</upper>
+          </limit>
+          <dynamics>
+            <damping>0.00001</damping>
+          </dynamics>
+				</axis>
+	    </joint>
+		</gazebo>
+  </xacro:macro>
 </robot>
