Commit message: added mimic tags in urdf

File: eeduro_delta_description/urdf/eeduro_delta.urdf.xacro (robot description, xacro)
@@ -172,4 +172,7 @@
 		  <axis xyz="1 0 0"/>
 		  <dynamics damping="0.00001"/>
+			<xacro:if value="${suffix == '_2'}">
+				<mimic joint="arm${arm_nr}_joint2_1" multiplier="1" offset="0"/>
+			</xacro:if>
 		</joint>
 		<link name="arm${arm_nr}_link3${suffix}">
@@ -185,5 +188,5 @@
 	</xacro:macro>
 	<xacro:macro name="joint3_urdf" params="arm_nr suffix">
-			<joint name="arm${arm_nr}_link3${suffix}" type="continuous">
+			<joint name="arm${arm_nr}_joint3${suffix}" type="continuous">
 			  <parent link="arm${arm_nr}_link3${suffix}"/>
 			  <child link="arm${arm_nr}_link4"/>
@@ -191,4 +194,5 @@
 			  <axis xyz="1 0 0"/>
 			  <dynamics damping="0.00001"/>
+				<mimic joint="arm${arm_nr}_joint2_1" multiplier="-1" offset="0"/>
 			</joint>
 	</xacro:macro>

Commit message: change initial position

File: eeduro_delta_description/urdf/eeduro_delta.urdf.xacro (robot description, xacro)
@@ -4,4 +4,7 @@
 	<xacro:property name="dist_origin2arm_z" value="0.21"/>
 	<xacro:property name="dist_origin2arm_xy_plane" value="${0.1/sqrt(3) -0.005}"/>
+	<xacro:property name="angle1_init" value="0.0"/>
+	<xacro:property name="angle2_init" value="-2.49368823859929645"/>
+	<xacro:property name="angle3_init" value="5.63528089218908956"/>
 	<xacro:include filename="$(find eeduro_delta_description)/urdf/eeduro_delta_inertial.urdf.xacro"/>
 	<!--<xacro:include filename="$(find eeduro_delta_description)/urdf/eeduro_delta.gazebo.xacro"/>-->
@@ -33,7 +36,7 @@
 		arm_nr="1"
 		joint4_type="urdf"
-		angle1="${(-27)/180.0*pi}"
-		angle2="${-0.8373228137897161 -(90-27)/180.0*pi}"
-		angle3="${-pi/2 + 0.8373228137897161}"
+		angle1="${angle1_init}"
+		angle2="${angle2_init}"
+		angle3="${angle3_init}"
 		dist_xy="${dist_origin2arm_xy_plane}"
 		x="0"		y="0"		z="${dist_origin2arm_z}"
@@ -45,7 +48,7 @@
     arm_nr="2"
     joint4_type="sdf"
-    angle1="${(-27)/180.0*pi}"
-    angle2="${-0.8373228137897161 -(90-27)/180.0*pi}"
-    angle3="${-pi/2 + 0.8373228137897161}"
+		angle1="${angle1_init}"
+		angle2="${angle2_init}"
+		angle3="${angle3_init}"
     dist_xy="${dist_origin2arm_xy_plane}"
     x="0"   y="0"   z="${dist_origin2arm_z}"
@@ -57,7 +60,7 @@
     arm_nr="3"
     joint4_type="sdf"
-    angle1="${(-27)/180.0*pi}"
-    angle2="${-0.8373228137897161 -(90-27)/180.0*pi}"
-    angle3="${-pi/2 + 0.8373228137897161}"
+		angle1="${angle1_init}"
+		angle2="${angle2_init}"
+		angle3="${angle3_init}"
     dist_xy="${dist_origin2arm_xy_plane}"
     x="0"   y="0"   z="${dist_origin2arm_z}"

Commit message: adjust joint_state_publisher for new inital position

File: eeduro_delta_description/urdf/eeduro_delta.urdf.xacro (robot description, xacro)
@@ -6,5 +6,5 @@
 	<xacro:property name="angle1_init" value="0.0"/>
 	<xacro:property name="angle2_init" value="-2.49368823859929645"/>
-	<xacro:property name="angle3_init" value="5.63528089218908956"/>
+	<xacro:property name="angle3_init" value="-0.64790441499049692"/>
 	<xacro:include filename="$(find eeduro_delta_description)/urdf/eeduro_delta_inertial.urdf.xacro"/>
 	<!--<xacro:include filename="$(find eeduro_delta_description)/urdf/eeduro_delta.gazebo.xacro"/>-->

Commit message: add collision to link1 and link2

File: eeduro_delta_description/urdf/eeduro_delta.urdf.xacro (robot description, xacro)
@@ -85,4 +85,22 @@
 	  <selfCollide>true</selfCollide>
 	</gazebo>
+	<gazebo reference="arm1_link1">
+	  <selfCollide>true</selfCollide>
+	</gazebo>
+	<gazebo reference="arm2_link1">
+	  <selfCollide>true</selfCollide>
+	</gazebo>
+	<gazebo reference="arm3_link1">
+	  <selfCollide>true</selfCollide>
+	</gazebo>
+	<gazebo reference="arm1_link2">
+	  <selfCollide>true</selfCollide>
+	</gazebo>
+	<gazebo reference="arm2_link2">
+	  <selfCollide>true</selfCollide>
+	</gazebo>
+	<gazebo reference="arm3_link2">
+	  <selfCollide>true</selfCollide>
+	</gazebo>
 	<gazebo reference="tool">
 	  <selfCollide>true</selfCollide>
@@ -121,4 +139,10 @@
 		    </geometry>
 		  </visual>
+			<collision>
+				<origin xyz="0 0 0.024" rpy="0 0 0"/>
+				<geometry>
+					<box size="0.006 0.012 0.06 "/>
+				</geometry>
+			</collision>
 			<xacro:link1_inertial/>
 		</link>
@@ -153,4 +177,10 @@
 		    </geometry>
 		  </visual>
+			<collision>
+		    <origin xyz="0 0 0" rpy="0 0 0"/>
+		    <geometry>
+					<box size="0.044 0.008 0.006"/>
+				</geometry>
+			</collision>
 			<xacro:link2_inertial/>
 		</link>

Commit message: add ros_control for 1 motor, not tested

File: eeduro_delta_description/urdf/eeduro_delta.urdf.xacro (robot description, xacro)
@@ -8,5 +8,5 @@
 	<xacro:property name="angle3_init" value="-0.64790441499049692"/>
 	<xacro:include filename="$(find eeduro_delta_description)/urdf/eeduro_delta_inertial.urdf.xacro"/>
-	<!--<xacro:include filename="$(find eeduro_delta_description)/urdf/eeduro_delta.gazebo.xacro"/>-->
+	<xacro:include filename="$(find eeduro_delta_description)/urdf/eeduro_delta.gazebo"/>
 	<link name="world"/>
 	<gazebo reference="world">
@@ -82,28 +82,14 @@
 		<xacro:tool_inertial/>
 	</link>
-	<gazebo reference="base_link">
-	  <selfCollide>true</selfCollide>
-	</gazebo>
-	<gazebo reference="arm1_link1">
-	  <selfCollide>true</selfCollide>
-	</gazebo>
-	<gazebo reference="arm2_link1">
-	  <selfCollide>true</selfCollide>
-	</gazebo>
-	<gazebo reference="arm3_link1">
-	  <selfCollide>true</selfCollide>
-	</gazebo>
-	<gazebo reference="arm1_link2">
-	  <selfCollide>true</selfCollide>
-	</gazebo>
-	<gazebo reference="arm2_link2">
-	  <selfCollide>true</selfCollide>
-	</gazebo>
-	<gazebo reference="arm3_link2">
-	  <selfCollide>true</selfCollide>
-	</gazebo>
-	<gazebo reference="tool">
-	  <selfCollide>true</selfCollide>
-	</gazebo>
+	<transmission name="tran1">
+		<type>transmission_interface/SimpleTransmission</type>
+		<joint name="arm1_joint0">
+			<hardwareInterface>hardware_interface/EffortJointInterface</hardwareInterface>
+		</joint>
+		<actuator name="motor1">
+			<hardwareInterface>hardware_interface/EffortJointInterface</hardwareInterface>
+			<mechanicalReduction>1</mechanicalReduction>
+		</actuator>
+	</transmission>
 	<!-- x y z are the center of the robot, in the high:of the mounting-points for the arms -->
 	<xacro:macro name="delta_arm" params="parent arm_end_child arm_nr joint4_type angle1 angle2 angle3 dist_xy x y z roll pitch yaw">
@@ -279,11 +265,3 @@
 		</gazebo>
   </xacro:macro>
-	<gazebo>
-		<plugin name="gazebo_ros_joint_state_publisher" filename="libgazebo_ros_joint_state_publisher.so">
-			<robotNamespace>/eeduro_delta</robotNamespace>
-			<jointName>arm1_joint0, arm2_joint0, arm3_joint0</jointName>
-			<updateRate>1000</updateRate>
-			<alwaysOn>true</alwaysOn>
-		</plugin>
-	</gazebo>
 </robot>
