Commit message: works with model 2

File: eeduro_delta_description/urdf/eeduro_delta2.urdf.xacro (robot description, xacro)
@@ -114,5 +114,5 @@
 	<!-- x y z are the center of the robot, in the high:of the mounting-points for the arms -->
 	<xacro:macro name="delta_arm" params="parent arm_end_child arm_nr joint4_type angle1 angle2 angle3 dist_xy x y z roll pitch yaw">
-		<joint name="arm${arm_nr}_motor_joint" type="continuous">
+<!--		<joint name="arm${arm_nr}_motor_joint" type="continuous">
 		  <parent link="${parent}"/>
 		  <child link="arm${arm_nr}_motor"/>
@@ -129,5 +129,5 @@
 	  </visual>
 		<xacro:motor_inertial/>
-		</link>
+		</link> -->
 		<joint name="arm${arm_nr}_joint0" type="continuous">
 		  <parent link="${parent}"/>
@@ -153,5 +153,5 @@
 			<xacro:link1_inertial/>
 		</link>
-		<gazebo>
+<!--		<gazebo>
 		  <joint name="arm${arm_nr}_gearbox" type="gearbox">
 		    <parent>arm${arm_nr}_motor</parent>
@@ -168,5 +168,5 @@
 		    </axis2>
 		  </joint>
-		</gazebo>
+		</gazebo> -->
 		<joint name="arm${arm_nr}_joint1" type="continuous">
 		  <parent link="arm${arm_nr}_link1"/>
